File: ADS1115_Grove_Emon.brd (EAGLE design)
At the start: 31.4 x 17.2 mm, 17 parts, among them J1 ST-PJ-312, J2 ST-PJ-312, J3 GROVE-4P-2.0-SMD-FEMALE-REINF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, J4 GROVE-4P-2.0-SMD-FEMALE-REINF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, U1 ADS1115IDGST

Commit message: v1 populated and routed
Parts:
- removed FID2: FIDUCIAL"", microbuilder:FIDUCIAL_1MM
- removed U$13, U$14: MOUNTINGHOLE2.5, microbuilder:MOUNTINGHOLE_2.5_PLATED
- added 0X48, 0X49, 0X4A, 0X4B: (no value), jumper:SJ
- added R5, R6: 100R, microbuilder:0603
- moved J4 6.60 mm to (32.5, 8.64)
- moved JP1 5.08 mm to (19.1, 1.65)
- moved J1 3.68 mm to (24.9, 20.3)
- moved J2 3.18 mm to (13.3, 20.3)
- moved U1 1.30 mm to (21.8, 10.7)
- moved C1 1.05 mm to (21.8, 13.2)
- moved J3 0.13 mm to (5.59, 8.64)
Connections:
- net ADDR: now also 0X48.1, 0X49.1, 0X4A.1, 0X4B.1
- net AIN0: now also J1.COM1, R6.1
- net AIN1: now also J1.L, R6.2
- net AIN2: now also J2.COM1, R5.1
- net AIN3: now also J2.L, R5.2
- net GND: now also 0X48.2, J3.1, J3.SS1, J3.SS2, J4.1, J4.SS1, J4.SS2
- net SCL: now also 0X4B.2, J3.4, J4.4
- net SDA: now also 0X4A.2, J3.3, J4.3
- net VDD: now also 0X49.2, J3.2, J4.2
Routing:
- net SDA: track 26.3 -> 60.4 mm, vias 1 -> 3
- net AIN2: track 7.02 -> 37.1 mm, vias 0 -> 2
- net GND: track 40.2 -> 11.0 mm, vias 0 -> 6
- net AIN3: track 13.5 -> 39.9 mm, vias 0 -> 1
- net ADDR: track 27.6 -> 49.9 mm, vias 1 -> 3
- net SCL: track 29.8 -> 48.8 mm, vias 1 -> 3
- net AIN0: track 8.23 -> 26.5 mm, vias 0 -> 1
- net VDD: track 32.2 -> 46.7 mm, vias 2 -> 3
- net AIN1: track 6.96 -> 21.1 mm, vias 0 -> 1
- net ALERT: track 12.4 -> 25.9 mm
- net N$2: track 8.39 -> 10.8 mm
- net N$1: track 8.32 -> 10.2 mm
Other:
- board size 31.4 x 17.2 mm -> 38.1 x 17.1 mm
- board text added: "04/12/2015 v1"
- board text added: "0x48"
- board text added: "0x49"
- board text added: "0x4A"
- board text added: "0x4B"
- board text added: "@whatnick"

Commit message: Fixed grove connector orientation
Parts:
- J3, J4: value GROVE-4P-2.0-SMD-FEMALE-REINFORCE-3470090P1 -> H4P-SMD-2.0; device OPL:4P-SMD-2.0 -> Seeed-OPL-Connector:HW4-SMD-2.0
- moved J4 26.8 mm to (5.71, 8.89), turned to 270 degrees
- moved J3 26.7 mm to (32.3, 8.51), turned to 90 degrees
Connections:
- new net 3V3: J3.3, J4.3
- net GND: now also J3.4, J4.4; no longer J3.1, J4.1
- net SCL: now also J3.1, J4.1; no longer J3.4, J4.4
- net SDA: now also J3.2, J4.2; no longer J3.3, J4.3
- net VDD: no longer J3.2, J4.2
Routing:
- net 3V3: track 0.00 -> 42.1 mm, vias 0 -> 2
- net AIN2: track 37.1 -> 75.0 mm, vias 2 -> 5
- net GND: track 11.0 -> 27.7 mm, vias 6 -> 8
- net SCL: track 48.8 -> 64.4 mm
- net VDD: track 46.7 -> 31.2 mm, vias 3 -> 2
- net AIN0: track 26.5 -> 41.3 mm, vias 1 -> 2
- net AIN3: track 39.9 -> 50.6 mm
- net SDA: track 60.4 -> 53.8 mm
- net ALERT: track 25.9 -> 19.7 mm, vias 0 -> 1
- net ADDR: track 49.9 -> 48.6 mm, vias 3 -> 5
- net AIN1: track 21.1 -> 20.2 mm
Other:
- board text added: "25/12/2015 v2"
- board text removed: "04/12/2015 v1"
