File: ADS1115_Grove_Emon.brd (EAGLE design)
At the start: 38.1 x 17.1 mm, 20 parts, among them J1 ST-PJ-312, J2 ST-PJ-312, J3 H4P-SMD-2.0, J4 H4P-SMD-2.0, U1 ADS1115IDGST

Commit message: Joined 3V3 to VDD
Connections:
- removed net 3V3: J3.3, J4.3
- net VDD: now also J3.3, J4.3
Routing:
- net 3V3: track 42.1 -> 0.00 mm, vias 2 -> 0
- net VDD: track 31.2 -> 73.2 mm, vias 2 -> 4
Changed lines of the file:
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@@
 <via x="22.70125" y="12.065" extent="1-16" drill="0.3302"/>
 <via x="19.05" y="12.3825" extent="1-16" drill="0.3302"/>
+<contactref element="J3" pad="3"/>
+<contactref element="J4" pad="3"/>
+<wire x1="2.54" y1="7.9375" x2="5.715" y2="7.9375" width="0.8128" layer="16"/>
+<wire x1="2.06375" y1="8.41375" x2="2.54" y2="7.9375" width="0.8128" layer="16"/>
+<wire x1="1.5875" y1="8.89" x2="2.06375" y2="8.41375" width="0.8128" layer="1"/>
+<wire x1="1.5875" y1="12.3825" x2="1.5875" y2="8.89" width="0.8128" layer="1"/>
+<wire x1="3.65125" y1="14.44625" x2="1.5875" y2="12.3825" width="0.8128" layer="1"/>
+<wire x1="24.60625" y1="14.44625" x2="3.65125" y2="14.44625" width="0.8128" layer="1"/>
+<wire x1="24.60625" y1="13.6525" x2="24.60625" y2="14.44625" width="0.8128" layer="1"/>
+<wire x1="27.6225" y1="10.63625" x2="24.60625" y2="13.6525" width="0.8128" layer="16"/>
+<wire x1="29.68625" y1="10.63625" x2="27.6225" y2="10.63625" width="0.8128" layer="16"/>
+<wire x1="30.1625" y1="10.16" x2="29.68625" y2="10.63625" width="0.8128" layer="16"/>
+<wire x1="30.48" y1="10.16" x2="30.1625" y2="10.16" width="0.8128" layer="16"/>
+<wire x1="31.115" y1="9.525" x2="30.48" y2="10.16" width="0.8128" layer="16"/>
+<wire x1="32.22625" y1="9.525" x2="31.115" y2="9.525" width="0.8128" layer="16"/>
+<wire x1="5.715" y1="7.9375" x2="5.715" y2="7.89" width="0.8128" layer="16"/>
+<via x="2.06375" y="8.41375" extent="1-16" drill="0.3302"/>
+<via x="24.60625" y="13.6525" extent="1-16" drill="0.3302"/>
+<wire x1="32.22625" y1="9.525" x2="32.258" y2="9.509" width="0" layer="19" extent="16-16"/>
+<wire x1="2.794" y1="11.518" x2="1.5875" y2="12.3825" width="0" layer="19" extent="1-1"/>
 </signal>
 <signal name="ALERT">
@@
 <wire x1="3.01625" y1="6.985" x2="2.96" y2="7.112" width="0.254" layer="1"/>
 </signal>
-<signal name="3V3" class="1">
-<contactref element="J3" pad="3"/>
-<contactref element="J4" pad="3"/>
-<wire x1="2.54" y1="7.9375" x2="5.715" y2="7.9375" width="0.8128" layer="16"/>
-<wire x1="2.06375" y1="8.41375" x2="2.54" y2="7.9375" width="0.8128" layer="16"/>
-<wire x1="1.5875" y1="8.89" x2="2.06375" y2="8.41375" width="0.8128" layer="1"/>
-<wire x1="1.5875" y1="12.3825" x2="1.5875" y2="8.89" width="0.8128" layer="1"/>
-<wire x1="3.65125" y1="14.44625" x2="1.5875" y2="12.3825" width="0.8128" layer="1"/>
-<wire x1="24.60625" y1="14.44625" x2="3.65125" y2="14.44625" width="0.8128" layer="1"/>
-<wire x1="24.60625" y1="13.6525" x2="24.60625" y2="14.44625" width="0.8128" layer="1"/>
-<wire x1="27.6225" y1="10.63625" x2="24.60625" y2="13.6525" width="0.8128" layer="16"/>
-<wire x1="29.68625" y1="10.63625" x2="27.6225" y2="10.63625" width="0.8128" layer="16"/>
-<wire x1="30.1625" y1="10.16" x2="29.68625" y2="10.63625" width="0.8128" layer="16"/>
-<wire x1="30.48" y1="10.16" x2="30.1625" y2="10.16" width="0.8128" layer="16"/>
-<wire x1="31.115" y1="9.525" x2="30.48" y2="10.16" width="0.8128" layer="16"/>
-<wire x1="32.22625" y1="9.525" x2="31.115" y2="9.525" width="0.8128" layer="16"/>
-<wire x1="5.715" y1="7.9375" x2="5.715" y2="7.89" width="0.8128" layer="16"/>
-<wire x1="32.22625" y1="9.525" x2="32.258" y2="9.509" width="0.8128" layer="16"/>
-<via x="2.06375" y="8.41375" extent="1-16" drill="0.3302"/>
-<via x="24.60625" y="13.6525" extent="1-16" drill="0.3302"/>
-</signal>
 </signals>

Commit message: Upped Version to v3
Routing:
- net VDD: track 73.2 -> 75.8 mm
Other:
- board text added: "17/01/2016 v3"
- board text removed: "25/12/2015 v2"
Changed lines of the file:
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@@
 <hole x="31.623" y="15.367" drill="1.27"/>
 <text x="36.068" y="8.636" size="1.016" layer="21" font="vector" ratio="20" rot="R270" align="center">@whatnick</text>
-<text x="35.052" y="2.921" size="1.016" layer="21" font="vector" ratio="20" rot="R90">25/12/2015 v2</text>
+<text x="35.052" y="2.921" size="1.016" layer="21" font="vector" ratio="20" rot="R90">17/01/2016 v3</text>
 </plain>
 <attributes>
@@
 <via x="2.06375" y="8.41375" extent="1-16" drill="0.3302"/>
 <via x="24.60625" y="13.6525" extent="1-16" drill="0.3302"/>
-<wire x1="32.22625" y1="9.525" x2="32.258" y2="9.509" width="0" layer="19" extent="16-16"/>
-<wire x1="2.794" y1="11.518" x2="1.5875" y2="12.3825" width="0" layer="19" extent="1-1"/>
+<wire x1="32.385" y1="9.525" x2="32.258" y2="9.509" width="0.254" layer="16"/>
+<wire x1="32.385" y1="9.525" x2="32.22625" y2="9.525" width="0.254" layer="16"/>
+<wire x1="22.86" y1="13.6525" x2="24.60625" y2="13.6525" width="0.6096" layer="1"/>
+<wire x1="22.86" y1="13.335" x2="22.86" y2="13.6525" width="0.254" layer="1"/>
+<wire x1="22.86" y1="13.335" x2="22.694" y2="13.208" width="0.254" layer="1"/>
 </signal>
 <signal name="ALERT">

Commit message: Rewired with 3V3 separated from VDD by ferrite
Parts:
- turned 0X48 to 180 degrees
- turned 0X4B to 180 degrees
Connections:
- removed net N$1: C2.1, FB1.1, JP1.10
- removed net N$2: C2.2, FB2.1, JP1.9
- new net 3V3: C2.1, FB1.1, J3.3, J4.3, JP1.10
- new net AGND: C2.2, FB2.1, J3.4, J4.4, JP1.9
- net GND: no longer J3.4, J4.4
- net VDD: no longer J3.3, J4.3
Routing:
- net AGND: track 0.00 -> 53.0 mm, vias 0 -> 1
- net 3V3: track 0.00 -> 42.1 mm, vias 0 -> 1
- net AIN2: track 75.0 -> 44.0 mm
- net GND: track 27.7 -> 55.2 mm, vias 8 -> 18
- net ADDR: track 48.6 -> 36.6 mm, vias 5 -> 0
- net N$2: track 10.8 -> 0.00 mm
- net N$1: track 10.2 -> 0.00 mm
- net AIN3: track 50.6 -> 40.8 mm, vias 1 -> 2
- net AIN0: track 41.3 -> 35.0 mm, vias 2 -> 1
- net SCL: track 64.4 -> 59.3 mm, vias 3 -> 4
- net ALERT: track 19.7 -> 15.5 mm, vias 1 -> 0
- net SDA: track 53.8 -> 57.7 mm, vias 3 -> 2
- net AIN1: track 20.2 -> 18.1 mm, vias 1 -> 2
- net VDD: track 75.8 -> 76.4 mm, vias 4 -> 2
